Commit message: fixed mobile robot navigation

File: src/td3/urdf/td_robot.urdf (robot description, URDF)
Before this commit: robot rs_robot, 17 links, 16 joints
Links:
- link chassis: geometry collision box size=0.225 0.220 0.108; visual box size=0.225 0.220 0.108
Joints:
- joint velodyne_base_mount_joint: origin xyz=0.125 0 0.25 rpy=0 0 0 -> xyz=0.125 0.02 0.25 rpy=0 0 0
