Commit message: updated sjtu

File: src/sjtu_drone/sjtu_drone_description/urdf/sjtu_drone.urdf.xacro (robot description, xacro)
@@ -22,14 +22,14 @@
     </inertial>
     <collision name="sjtu_drone_collision">
-      <origin rpy="0 0 0" xyz="0   0   0.04"/>
+      <origin rpy="0 0 0" xyz="0   0   -0.04"/>
       <geometry>
-        <mesh filename="file://$(find sjtu_drone_description)/models/sjtu_drone/quadrotor_4.stl"/>
+        <mesh filename="file://$(find sjtu_drone_description)/models/F450/F450.dae"/>
         <!-- <mesh filename="package://sjtu_drone/quadrotor_4.stl"/> -->
       </geometry>
     </collision>
     <visual name="sjtu_drone_visual">
-      <origin rpy="0 0 0" xyz="0   0   0.04"/>
+      <origin rpy="0 0 0" xyz="0   0   -0.04"/>
       <geometry>
-        <mesh filename="file://$(find sjtu_drone_description)/models/sjtu_drone/quadrotor_4.dae"/>
+        <mesh filename="file://$(find sjtu_drone_description)/models/F450/F450.dae"/>
         <!-- <mesh filename="package://sjtu_drone/quadrotor_4.dae"/> -->
       </geometry>
@@ -183,5 +183,5 @@
       </gazebo>
     <joint name="rplidar_link_joint" type="fixed">
-        <origin rpy="0 0 0" xyz="0.0 0 0.13"/>
+        <origin rpy="0 0 0" xyz="0.0 0 0.075"/>
         <parent link="base_link"/>
         <child link="lidar_link"/>
